File: Testing/Testing Emiliano/PCB_REGULADOR_SOLAR/pcb_regulador_solar_V1.0/pcb_regulador_solar_V1.0.sch (KiCad schematic (older format))
At the start: 2 parts

Commit message: Avance PCB Regulador solar
Parts:
- removed U?: INA219AxD, Package_SO:SOIC-8_3.9x4.9mm_P1.27mm, symbol Analog_ADC:INA219AxD
- removed U?: ESP32_NODEMCU, MODULE_ESP32_NODEMCU, symbol ESP32_NODEMCU:ESP32_NODEMCU
- added Q1 (x5): BC337, Package_TO_SOT_THT:TO-92_Inline, symbol Transistor_BJT:BC337
- added Q2 (x3): BC327, Package_TO_SOT_THT:TO-92_Inline, symbol Transistor_BJT:BC327
- added Q3 (x4): IRF4905, Package_TO_SOT_THT:TO-220-3_Vertical, symbol Transistor_FET:IRF4905
- added R1 (x9): 10k, symbol Device:R
- added R2: 1k, symbol Device:R
- added R3: 3k9, symbol Device:R
Connections:
- net labels added: GND
- wire segments 0 -> 39
