File: Testing/Testing Emiliano/PCB_REGULADOR_SOLAR/pcb_regulador_solar_V1.0/pcb_regulador_solar_V1.0.sch (KiCad schematic (older format))
At the start: 2 parts

Commit message: HArvest energy clone
Parts:
- added J?: Conn_01x06_MountingPin, symbol Connector_Generic_MountingPin:Conn_01x06_MountingPin
Connections:
- net at U?.J5_18 (EN): now also J?.6 (Pin_6)
Changed lines of the file:
@@
 	1    0    0    -1
 $EndComp
+$Comp
+L Connector_Generic_MountingPin:Conn_01x06_MountingPin J?
+U 1 1 644AF62C
+P 2900 1250
+F 0 "J?" H 2988 1164 50  0000 L CNN
+F 1 "Conn_01x06_MountingPin" H 2988 1073 50  0000 L CNN
+F 2 "" H 2900 1250 50  0001 C CNN
+F 3 "~" H 2900 1250 50  0001 C CNN
+	1    2900 1250
+	1    0    0    -1
+$EndComp
+Wire Wire Line
+	4500 1850 2700 1850
+Wire Wire Line
+	2700 1850 2700 1550
 $EndSCHEMATC
