File: Testing/Testing Emiliano/PCB_REGULADOR_SOLAR/pcb_regulador_solar_V1.0/pcb_regulador_solar_V1.0.kicad_sch (KiCad schematic)
At the start: 54 parts, among them J1 Conn_01x03_Pin, J2 Screw_Terminal_01x02, Q1 BC557, Q2 BC557, Q3 2N3904, Q4 2N3904, Q5 2N3904, Q6 IRF4905, SW1 RESET MANUAL, U1 PC817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

Commit message: Etapa entrada
Parts:
- added C10: 100n, symbol Device:C
- added C9: 1000u 25v, symbol Device:C_Polarized
- added D9: 1N5822, Diode_THT:D_DO-201AD_P15.24mm_Horizontal, symbol Diode:1N5822
- added R25: 0,1 (2w), symbol Device:R
- added U5: INA219AxD, Package_TO_SOT_SMD:SOT-23-8, symbol Sensor_Energy:INA219AxD
Connections:
- net +3.3V: now also U5.5 (VS)
- net GND: now also C10.2, C9.2, U5.6 (GND)
- new net: C10.1, C9.1, R25.2, U5.7 (IN-)
- new net: D9.1 (K), R25.1, U5.8 (IN+)
Other:
- moved on the sheet: C1, C2, C3, C4, C5, C6, C7, C8, D1, D10, D2, D3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
