File: Testing/Testing Emiliano/PCB_REGULADOR_SOLAR/pcb_regulador_solar_V1.0/pcb_regulador_solar_V1.0.kicad_sch (KiCad schematic)
At the start: 59 parts, among them J1 Conn_01x03_Pin, J2 Screw_Terminal_01x02, Q1 BC557, Q2 BC557, Q3 2N3904, Q4 2N3904, Q5 2N3904, Q6 IRF4905, SW1 RESET MANUAL, U1 PC817, U2 NE555P, U3 PC817, U4 LM358, U5 INA219AxD

Commit message: Avance PCB UPS
Parts:
- removed U5: INA219AxD, Package_TO_SOT_SMD:SOT-23-8, symbol Sensor_Energy:INA219AxD
- added C11, C16, C17, C18, C21: 100nf, Capacitor_THT:C_Axial_L5.1mm_D3.1mm_P7.50mm_Horizontal, symbol Device:C
- added C12, C13: 100n, Capacitor_THT:C_Axial_L5.1mm_D3.1mm_P7.50mm_Horizontal, symbol Device:C
- added C14: 100u 25v, Capacitor_THT:C_Radial_D5.0mm_H11.0mm_P2.00mm, symbol Device:C_Polarized
- added C15, C19, C20: 10nf, Capacitor_THT:C_Axial_L5.1mm_D3.1mm_P7.50mm_Horizontal, symbol Device:C
- added C22: 22u 25v, Capacitor_THT:C_Radial_D5.0mm_H11.0mm_P2.00mm, symbol Device:C_Polarized
- added C23: 47u 16v, Capacitor_THT:C_Radial_D5.0mm_H11.0mm_P2.00mm, symbol Device:C_Polarized
- added D11, D17, D22: LED VERDE, symbol Device:LED
- added D12: 1.5KE30A, Diode_THT:D_DO-201AE_P15.24mm_Horizontal, symbol Diode:1.5KExxA
- added D13, D15, D16, D23: 18v, symbol Device:D_Zener
- added D14, D18, D19, D24, D25, D28: 1N5819, Diode_THT:D_DO-41_SOD81_P10.16mm_Horizontal, symbol Diode:1N5819
- added D20: 1.5KE18, Diode_THT:D_DO-201AE_P15.24mm_Horizontal, symbol Diode:1.5KExxA
- added D21, D26: 3.3, symbol Device:D_Zener
- added D27: LED ROJO, symbol Device:LED
- added DCDC1, DCDC5: IN-, symbol Connector:Conn_01x01_Pin
- added DCDC2, DCDC6: OUT+, symbol Connector:Conn_01x01_Pin
- added DCDC3, DCDC7: OUT-, symbol Connector:Conn_01x01_Pin
- added DCDC4, DCDC8: IN+, symbol Connector:Conn_01x01_Pin
- added F1, F2: Fuse 3A, symbol Device:Fuse
- added J10: Conn_01x03_Pin, symbol Connector:Conn_01x03_Pin
- added J3, J9: INA219, symbol Connector:Conn_01x06_Pin
- added J4: Conn_01x02_Pin, symbol Connector:Conn_01x02_Pin
- added J5, J7, J8: Screw_Terminal_01x02, symbol Connector:Screw_Terminal_01x02
- added J6: USB_A, symbol Connector:USB_A
- added LEFT_ESP1: L ESP, symbol Connector:Conn_01x15_Pin
- added Q10, Q17, Q18, Q20, Q21, Q22: 2N3904, Package_TO_SOT_THT:TO-92_Inline, symbol Transistor_BJT:2N3904
- added Q11, Q8: IRLIZ44N, Package_TO_SOT_THT:TO-220F-3_Vertical, symbol Transistor_FET:IRLIZ44N
- added Q12, Q14, Q19, Q7: IRF4905, Package_TO_SOT_THT:TO-220-3_Vertical, symbol Transistor_FET:IRF4905
- added Q13: 2N7000, Package_TO_SOT_THT:TO-92_Inline, symbol Transistor_FET:2N7000
- added Q15: BC337, Package_TO_SOT_THT:TO-92_Inline, symbol Transistor_BJT:BC337
- added Q16: BC327, Package_TO_SOT_THT:TO-92_Inline, symbol Transistor_BJT:BC327
- added Q23, Q24, Q9: BC557, Package_TO_SOT_THT:TO-92_Inline, symbol Transistor_BJT:BC557
- added R26, R31, R46, R47, R48: 0,1 (2w), Resistor_THT:R_Axial_DIN0207_L6.3mm_D2.5mm_P2.54mm_Vertical, symbol Device:R
- added R27, R32, R33, R34, R45, R51, R53, R55, R64, R68, R70, R74, R75, R76, R78: 10k, Resistor_THT:R_Axial_DIN0207_L6.3mm_D2.5mm_P2.54mm_Vertical, symbol Device:R
- added R28, R38, R61: 470k, Resistor_THT:R_Axial_DIN0207_L6.3mm_D2.5mm_P2.54mm_Vertical, symbol Device:R
- added R29, R36, R39, R41, R49, R63: 10, Resistor_THT:R_Axial_DIN0207_L6.3mm_D2.5mm_P2.54mm_Vertical, symbol Device:R
- added R30, R37, R40, R65: 220, Resistor_THT:R_Axial_DIN0207_L6.3mm_D2.5mm_P2.54mm_Vertical, symbol Device:R
- added R35, R52, R54, R79: 100k, Resistor_THT:R_Axial_DIN0207_L6.3mm_D2.5mm_P2.54mm_Vertical, symbol Device:R
- added R42, R43, R44, R67: 1M, Resistor_THT:R_Axial_DIN0207_L6.3mm_D2.5mm_P2.54mm_Vertical, symbol Device:R
- added R50: 3.9K, Resistor_THT:R_Axial_DIN0207_L6.3mm_D2.5mm_P2.54mm_Vertical, symbol Device:R
- added R56, R59, R62: 220k (1%), Resistor_THT:R_Axial_DIN0207_L6.3mm_D2.5mm_P2.54mm_Vertical, symbol Device:R
- added R57: 0.1 (0.5W), Resistor_THT:R_Axial_DIN0207_L6.3mm_D2.5mm_P2.54mm_Vertical, symbol Device:R
- added R58: 47k (1%), Resistor_THT:R_Axial_DIN0207_L6.3mm_D2.5mm_P2.54mm_Vertical, symbol Device:R
- added R60: 10k (1%), Resistor_THT:R_Axial_DIN0207_L6.3mm_D2.5mm_P2.54mm_Vertical, symbol Device:R
- added R66, R69, R71: 220k, Resistor_THT:R_Axial_DIN0207_L6.3mm_D2.5mm_P2.54mm_Vertical, symbol Device:R
- added R72, R73: 1k, Resistor_THT:R_Axial_DIN0207_L6.3mm_D2.5mm_P2.54mm_Vertical, symbol Device:R
- added R77: 47k, Resistor_THT:R_Axial_DIN0207_L6.3mm_D2.5mm_P2.54mm_Vertical, symbol Device:R
- added RIGHT_ESP1: R ESP, symbol Connector:Conn_01x15_Pin
- added SW2, SW3: RESET MANUAL, symbol Switch:SW_SPST
- added unit 3 of U4
- added U5: LM358, Package_DIP:DIP-8_W7.62mm, symbol Amplifier_Operational:LM358
- added U6, U8: PC817, Package_DIP:DIP-4_W7.62mm, symbol Isolator:PC817
- added U7: NE555P, Package_DIP:DIP-8_W7.62mm, symbol Timer:NE555P
- C1, C10, C2, C5, C6, C7, C8: footprint (none) -> Capacitor_THT:C_Axial_L5.1mm_D3.1mm_P7.50mm_Horizontal
- C3, C4: footprint (none) -> Capacitor_THT:C_Radial_D5.0mm_H11.0mm_P2.00mm
- C9: footprint (none) -> Capacitor_THT:C_Radial_D10.0mm_H20.0mm_P5.00mm
- R1, R10, R11, R14, R15, R16, R17, R2, R20, R21, R22, R23, R24, R25, R3, R4, R5, R6, R7, R8, R9: footprint (none) -> Resistor_THT:R_Axial_DIN0207_L6.3mm_D2.5mm_P2.54mm_Vertical
- R12: value 220k -> 220; footprint (none) -> Resistor_THT:R_Axial_DIN0207_L6.3mm_D2.5mm_P2.54mm_Vertical
- R13: value 10k -> 10; footprint (none) -> Resistor_THT:R_Axial_DIN0207_L6.3mm_D2.5mm_P2.54mm_Vertical
- R18: value 220k -> 0.1 (0.5W); footprint (none) -> Resistor_THT:R_Axial_DIN0207_L6.3mm_D2.5mm_P2.54mm_Vertical
- R19: value 470k -> 47k (1%); footprint (none) -> Resistor_THT:R_Axial_DIN0207_L6.3mm_D2.5mm_P2.54mm_Vertical
Connections:
- net +3.3V: now also D25.2 (A), J3.6 (Pin_6), J9.6 (Pin_6), RIGHT_ESP1.1 (Pin_1)
- net +5V: now also C11.2, C17.2, C21.2, DCDC6.1 (Pin_1), J10.1 (Pin_1), LEFT_ESP1.15 (Pin_15), Q7.3 (S), Q9.3 (E), R33.2, R71.2, R72.1, R77.1, SW2.1 (A), U4.8 (V+), U5.8 (V+), U6.4, U7.4 (R), U7.8 (VCC)
- net GND: now also R18.2, C11.1, C12.2, C13.2, C14.2, C15.1, C16.1, C17.1, C18.1, C19.2, C20.2, C21.1, C22.2, D13.2 (A), D16.2 (A), D21.2 (A), D26.2 (A), DCDC1.1 (Pin_1), DCDC3.1 (Pin_1), DCDC5.1 (Pin_1), DCDC7.1 (Pin_1), J3.5 (Pin_5), J6.4 (GND), J6.5 (Shield), J9.5 (Pin_5), LEFT_ESP1.14 (Pin_14), Q10.1 (E), Q11.3 (S), Q13.1 (S), Q16.1 (C), Q17.1 (E), Q18.1 (E), Q20.1 (E), Q21.1 (E), Q22.1 (E), Q24.1 (C), Q8.3 (S), R28.2, R32.1, R35.1, R38.2, R43.2, R52.1, R54.1, R57.2, R58.1, R60.1, R61.2, R67.2, R76.1, R78.1, R79.1, U4.4 (V-), U5.4 (V-), U6.2, U7.1 (GND)
- net VCC: now also C10.1, C9.1, R25.2, DCDC4.1 (Pin_1), J10.3 (Pin_3), J3.2 (Pin_2), Q14.3 (S), Q15.1 (C), R26.2, R31.2, R44.2, R51.2
- net at C5.2, D10.1 (A1), D5.1 (K)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: now also R56.1; no longer R18.2
- net at D9.1 (K), R25.1: now also J3.1 (Pin_1), R26.1, R31.1
- net at D9.2 (A): now also J4.1 (Pin_1)
- net ADC V renamed ADC V1
- net ADC V1: now also LEFT_ESP1.2 (Pin_2), R56.2; no longer R18.1
- net ON/OFF renamed ON/OFF 1
- net ON/OFF 1: now also RIGHT_ESP1.15 (Pin_15)
- net PIN DIGITAL MICRO renamed ALARMA SC 1
- net ALARMA SC 1: now also RIGHT_ESP1.6 (Pin_6)
- new net: Q15.2 (B), Q16.2 (B), R50.1
- new net: Q15.3 (E), Q16.3 (E), R49.2
- new net: Q17.3 (C), R50.2, R51.1
- new net: J9.1 (Pin_1), Q12.2 (D), R46.1, R47.1, R48.1
- new net: D17.2 (A), J9.2 (Pin_2), Q14.2 (D), R46.2, R47.2, R48.2
- new net: R68.1, R69.1, R70.2, U7.7 (DIS), U8.4
- new net: Q20.2 (B), R68.2
- new net: Q10.3 (C), R27.1, R33.1
- new net: Q9.2 (B), R27.2
- new net: D13.1 (K), R29.2, R30.1
- new net: C12.1, D11.2 (A), D12.1 (A1), DCDC8.1 (Pin_1), F1.2, R30.2
- new net: Q24.2 (B), R75.2
- new net: D27.1 (K), Q24.3 (E)
- new net: D23.1 (K), J10.2 (Pin_2), Q19.3 (S), R66.1
- new net: D23.2 (A), R63.2, R65.2, R66.2
- new net: Q18.2 (B), R54.2, R55.2
- new net: Q18.3 (C), R41.2, R43.1, R44.1, R45.1
- new net: R69.2, U6.3
- new net: R72.2, U8.1
- new net: C18.2, Q22.3 (C), R67.1, U7.2 (TR), U8.2
- new net: C22.1, Q21.3 (C), R71.1, U8.3
- new net: C19.1, U7.5 (CV)
- new net: Q11.1 (G), R36.1
- new net: D16.1 (K), R36.2, R37.1
- new net: R60.2, R62.1, U5.2 (-)
- new net: J7.1 (Pin_1), Q11.2 (D)
- new net: Q17.2 (B), R52.2, R53.2
- new net: C23.1, D28.1 (K), R78.2, SW2.2 (B)
- new net: C23.2, D24.2 (A), R73.1, R76.2
- new net: D22.1 (K), R61.1
- new net: C16.2, D20.1 (A1), D22.2 (A), D24.1 (K), J8.2 (Pin_2), Q19.2 (D), R59.1, R64.2
- new net: R74.1, R75.1, U7.3 (Q)
- new net: D11.1 (K), R28.1
- new net: C15.2, D20.2 (A2), J8.1 (Pin_1), R18.1, R57.1, U5.3 (+)
- new net: Q10.2 (B), R34.2, R35.2
- new net: R64.1, U6.1
- new net: D12.2 (A2), J5.1 (Pin_1), Q8.2 (D)
- new net: F1.1, J5.2 (Pin_2)
- new net: C20.1, R62.2, U5.1, U7.6 (THR)
- new net: D18.1 (K), R53.1
- new net: Q22.2 (B), R73.2
- new net: D25.1 (K), Q23.3 (E)
- new net: DCDC2.1 (Pin_1), J4.2 (Pin_2)
- new net: Q23.2 (B), R74.2
- new net: D14.1 (K), R34.1
- new net: D27.2 (A), R77.2
- new net: Q20.3 (C), R65.1
- new net: Q19.1 (G), R63.1
- new net: Q12.1 (G), R39.1
- new net: C13.1, C14.1, D15.1 (K), F2.2, Q12.3 (S), R37.2, R42.1, SW3.1 (A)
- new net: J6.1 (VBUS), Q7.2 (D)
- new net: D17.1 (K), R38.1
- new net: Q14.1 (G), R49.1
- new net: D19.1 (K), R55.1
- new net: Q8.1 (G), R29.1
- new net: F2.1, J7.2 (Pin_2)
- new net: Q21.2 (B), R70.1
- new net: D15.2 (A), R39.2, R40.1, R42.2
- new net: Q13.3 (D), R40.2
- new net: Q7.1 (G), Q9.1 (C), R32.2
- new net: R45.2, SW3.2 (B)
- new net: Q13.2 (G), R41.1
- new net ADC V2: D21.1 (K), LEFT_ESP1.3 (Pin_3), R58.2, R59.2
- new net ALARMA SC 2: D26.1 (K), Q23.1 (C), R79.2, RIGHT_ESP1.5 (Pin_5)
- new net CORTE BAT: D19.2 (A), RIGHT_ESP1.7 (Pin_7)
- new net ON/OFF 2: D28.2 (A), RIGHT_ESP1.10 (Pin_10)
- new net PWM: D18.2 (A), RIGHT_ESP1.9 (Pin_9)
- new net RESET MODEM: D14.2 (A), LEFT_ESP1.6 (Pin_6)
- new net SCL: J3.4 (Pin_4), J9.4 (Pin_4), RIGHT_ESP1.14 (Pin_14)
- new net SDA: J3.3 (Pin_3), J9.3 (Pin_3), RIGHT_ESP1.11 (Pin_11)
Other:
- note added: "GND"
- note added: "SCL"
- note added: "SDA"
- note added: "VCC"
- note added: "Vin+"
- note added: "Vin-"
- moved on the sheet: C1, C2, C3, C4, C5, C6, C7, C8, D1, D10, D2, D3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

Commit message: pcb sOLAR
Parts:
- removed SW1, SW2, SW3: RESET MANUAL, symbol Switch:SW_SPST
- added SW1, SW2, SW4: RESET MANUAL, Button_Switch_SMD:SW_SPST_CK_RS282G05A3, symbol Switch:SW_Push
- D11, D17, D22, D27, D4, D7: footprint (none) -> LED_THT:LED_D3.0mm_IRBlack
- D13, D15, D16, D21, D23, D26, D3, D6, D8: footprint (none) -> Diode_THT:D_DO-35_SOD27_P7.62mm_Horizontal
- DCDC1, DCDC2, DCDC3, DCDC4, DCDC5, DCDC6, DCDC7, DCDC8: footprint (none) -> Connector_PinHeader_2.54mm:PinHeader_1x01_P2.54mm_Vertical
- F1, F2: footprint (none) -> Fuse:Fuseholder_Clip-5x20mm_Bel_FC-203-22_Lateral_P17.80x5.00mm_D1.17mm_Horizontal
- J1, J10: footprint (none) -> Connector_PinHeader_2.54mm:PinHeader_1x03_P2.54mm_Vertical
- J2, J5, J7, J8: footprint (none) -> TerminalBlock:TerminalBlock_bornier-3_P5.08mm
- J3, J9: footprint (none) -> Connector_PinSocket_2.54mm:PinSocket_1x06_P2.54mm_Vertical
- J4: footprint (none) -> Connector_PinHeader_2.54mm:PinHeader_1x02_P2.54mm_Vertical
- J6: footprint (none) -> Connector_USB:USB_A_Wuerth_614004134726_Horizontal
- LEFT_ESP1, RIGHT_ESP1: footprint (none) -> Connector_PinSocket_2.54mm:PinSocket_1x15_P2.54mm_Vertical
Connections:
- net +5V: now also SW1.2, SW4.2
- net at C23.1, D28.1 (K), R78.2: now also SW1.1
- net at C3.1, D1.1 (K), R5.2: now also SW4.1
- net at C13.1, C14.1, D15.1 (K)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: now also SW2.2
- net at R45.2: now also SW2.1

Commit message: Armado PCB
Parts:
- J2, J5, J7, J8: footprint TerminalBlock:TerminalBlock_bornier-3_P5.08mm -> TerminalBlock:TerminalBlock_bornier-2_P5.08mm
Changed lines of the file:
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@@
       (effects (font (size 1.27 1.27)))
     )
-    (property "Footprint" "TerminalBlock:TerminalBlock_bornier-3_P5.08mm" (at 281.94 260.35 0)
+    (property "Footprint" "TerminalBlock:TerminalBlock_bornier-2_P5.08mm" (at 281.94 260.35 0)
       (effects (font (size 1.27 1.27)) hide)
     )
@@
       (effects (font (size 1.27 1.27)))
     )
-    (property "Footprint" "TerminalBlock:TerminalBlock_bornier-3_P5.08mm" (at 73.66 34.29 0)
+    (property "Footprint" "TerminalBlock:TerminalBlock_bornier-2_P5.08mm" (at 73.66 34.29 0)
       (effects (font (size 1.27 1.27)) hide)
     )
@@
       (effects (font (size 1.27 1.27)))
     )
-    (property "Footprint" "TerminalBlock:TerminalBlock_bornier-3_P5.08mm" (at 72.39 77.47 0)
+    (property "Footprint" "TerminalBlock:TerminalBlock_bornier-2_P5.08mm" (at 72.39 77.47 0)
       (effects (font (size 1.27 1.27)) hide)
     )
@@
       (effects (font (size 1.27 1.27)))
     )
-    (property "Footprint" "TerminalBlock:TerminalBlock_bornier-3_P5.08mm" (at 46.99 264.16 0)
-      (effects (font (size 1.27 1.27)) hide)
-    )
+    (property "Footprint" "TerminalBlock:TerminalBlock_bornier-2_P5.08mm" (at 46.99 264.16 0)
+      (effects (font (size 1.27 1.27)) hide)
+    )

Commit message: actualizacion pcb_regulador_solar
Parts:
- removed C18, C21: 100nf, Capacitor_THT:C_Axial_L5.1mm_D3.1mm_P7.50mm_Horizontal, symbol Device:C
- removed C19, C20, C6: 10nf, Capacitor_THT:C_Axial_L5.1mm_D3.1mm_P7.50mm_Horizontal, symbol Device:C
- removed C22: 22u 25v, Capacitor_THT:C_Radial_D5.0mm_H11.0mm_P2.00mm, symbol Device:C_Polarized
- removed C23: 47u 16v, Capacitor_THT:C_Radial_D5.0mm_H11.0mm_P2.00mm, symbol Device:C_Polarized
- removed D13, D15, D16, D23, D6: 18v, Diode_THT:D_DO-35_SOD27_P7.62mm_Horizontal, symbol Device:D_Zener
- removed D17, D22: LED VERDE, LED_THT:LED_D3.0mm_IRBlack, symbol Device:LED
- removed D19, D2, D25, D28: 1N5819, Diode_THT:D_DO-41_SOD81_P10.16mm_Horizontal, symbol Diode:1N5819
- removed D20: 1.5KE18, Diode_THT:D_DO-201AE_P15.24mm_Horizontal, symbol Diode:1.5KExxA
- removed D21, D26, D3, D8: 3.3, Diode_THT:D_DO-35_SOD27_P7.62mm_Horizontal, symbol Device:D_Zener
- removed D27: LED ROJO, LED_THT:LED_D3.0mm_IRBlack, symbol Device:LED
- removed D9: 1N5822, Diode_THT:D_DO-201AD_P15.24mm_Horizontal, symbol Diode:1N5822
- removed J10: Conn_01x03_Pin, Connector_PinHeader_2.54mm:PinHeader_1x03_P2.54mm_Vertical, symbol Connector:Conn_01x03_Pin
- removed J4: Conn_01x02_Pin, Connector_PinHeader_2.54mm:PinHeader_1x02_P2.54mm_Vertical, symbol Connector:Conn_01x02_Pin
- removed J8: Screw_Terminal_01x02, TerminalBlock:TerminalBlock_bornier-2_P5.08mm, symbol Connector:Screw_Terminal_01x02
- removed Q1, Q2, Q23, Q24: BC557, Package_TO_SOT_THT:TO-92_Inline, symbol Transistor_BJT:BC557
- removed Q10, Q17, Q18, Q20, Q21, Q22, Q3, Q4, Q5: 2N3904, Package_TO_SOT_THT:TO-92_Inline, symbol Transistor_BJT:2N3904
- removed Q13: 2N7000, Package_TO_SOT_THT:TO-92_Inline, symbol Transistor_FET:2N7000
- removed Q19: IRF4905, Package_TO_SOT_THT:TO-220-3_Vertical, symbol Transistor_FET:IRF4905
- removed R65: 220, Resistor_THT:R_Axial_DIN0207_L6.3mm_D2.5mm_P2.54mm_Vertical, symbol Device:R
- removed R66, R69, R71: 220k, Resistor_THT:R_Axial_DIN0207_L6.3mm_D2.5mm_P2.54mm_Vertical, symbol Device:R
- removed R67: 1M, Resistor_THT:R_Axial_DIN0207_L6.3mm_D2.5mm_P2.54mm_Vertical, symbol Device:R
- removed R68, R70, R74, R75, R76, R78: 10k, Resistor_THT:R_Axial_DIN0207_L6.3mm_D2.5mm_P2.54mm_Vertical, symbol Device:R
- removed R72, R73: 1k, Resistor_THT:R_Axial_DIN0207_L6.3mm_D2.5mm_P2.54mm_Vertical, symbol Device:R
- removed R77: 47k, Resistor_THT:R_Axial_DIN0207_L6.3mm_D2.5mm_P2.54mm_Vertical, symbol Device:R
- removed R79: 100k, Resistor_THT:R_Axial_DIN0207_L6.3mm_D2.5mm_P2.54mm_Vertical, symbol Device:R
- removed SW2: RESET MANUAL, Button_Switch_SMD:SW_SPST_CK_RS282G05A3, symbol Switch:SW_Push
- removed U3, U6, U8: PC817, Package_DIP:DIP-4_W7.62mm, symbol Isolator:PC817
- removed U4, U5: LM358, Package_DIP:DIP-8_W7.62mm, symbol Amplifier_Operational:LM358
- removed U7: NE555P, Package_DIP:DIP-8_W7.62mm, symbol Timer:NE555P
- added ACS1, ACS4: OUT, Connector_PinHeader_2.54mm:PinHeader_1x01_P2.54mm_Vertical, symbol Connector:Conn_01x01_Pin
- added ACS2, ACS712: IN-, Connector_PinHeader_2.54mm:PinHeader_1x01_P2.54mm_Vertical, symbol Connector:Conn_01x01_Pin
- added ACS3, ACS712: Vcc, Connector_PinHeader_2.54mm:PinHeader_1x01_P2.54mm_Vertical, symbol Connector:Conn_01x01_Pin
- added ACS5, ACS712: IN+, Connector_PinHeader_2.54mm:PinHeader_1x01_P2.54mm_Vertical, symbol Connector:Conn_01x01_Pin
- added ACS6, ACS712: GND, Connector_PinHeader_2.54mm:PinHeader_1x01_P2.54mm_Vertical, symbol Connector:Conn_01x01_Pin
- added C18: 22u 16v, Capacitor_THT:C_Radial_D5.0mm_H11.0mm_P2.00mm, symbol Device:C_Polarized
- added C19: 47u 16v, Capacitor_THT:C_Radial_D5.0mm_H11.0mm_P2.00mm, symbol Device:C_Polarized
- added C6: 1u 16V, Capacitor_THT:C_Radial_D5.0mm_H11.0mm_P2.00mm, symbol Device:C_Polarized
- added D13, D16, D17, D19, D20, D21, D29, D30, D33, D6, D8, D9: 1N4746A, Diode_THT:D_DO-41_SOD81_P10.16mm_Horizontal, symbol Diode:1N47xxA
- added D15, D3: LED VERDE, LED_THT:LED_D3.0mm_IRBlack, symbol Device:LED
- added D2: 1.5KE18, Diode_THT:D_DO-201AE_P15.24mm_Horizontal, symbol Diode:1.5KExxA
- added D22, D31, D32: 1N5819, Diode_THT:D_DO-41_SOD81_P10.16mm_Horizontal, symbol Diode:1N5819
- added D23: LED ROJO, LED_THT:LED_D3.0mm_IRBlack, symbol Device:LED
- added D34: LED AZUL, LED_THT:LED_D3.0mm_IRBlack, symbol Device:LED
- added J4: OUT 2, TerminalBlock:TerminalBlock_bornier-2_P5.08mm, symbol Connector:Screw_Terminal_01x02
- added Q1, Q10, Q13, Q17, Q18, Q19, Q2, Q4, Q5: BC546, Package_TO_SOT_THT:TO-92_Inline, symbol Transistor_BJT:BC546
- added Q3: IRF4905, Package_TO_SOT_THT:TO-220-3_Vertical, symbol Transistor_FET:IRF4905
- added R80: 100k, Resistor_THT:R_Axial_DIN0207_L6.3mm_D2.5mm_P2.54mm_Vertical, symbol Device:R
- added SENSOR_TEMP: Conn_01x03_Pin, Connector_PinHeader_2.54mm:PinHeader_1x03_P2.54mm_Vertical, symbol Connector:Conn_01x03_Pin
- added U3: NE555P, Package_DIP:DIP-8_W7.62mm, symbol Timer:NE555P
- added U4: PC817, Package_DIP:DIP-4_W7.62mm, symbol Isolator:PC817
- C11, C8: value 100nf -> 100n
- C13: value 100n -> 100nf
- C14: value 100u 25v -> 1u 16V
- C17: value 100nf -> 10nf
- C4: value 22u 25v -> 22u 16v
- C9: value 1000u 25v -> 470u 50v
- F1, F2: value Fuse 3A -> Fuse 10A
- J2: value Screw_Terminal_01x02 -> OUT 1
- Q11, Q8: value IRLIZ44N -> IRFZ44N
- R12, R30, R37: value 220 -> 220 (1W)
- R13: value 10 -> 1M
- R16: value 10k -> 3.9 k
- R17: value 470k -> 22k
- R18: value 0.1 (0.5W) -> 3.9 k
- R2: value 100k -> 15k
- R20: value 0.1 (0.5W) -> 47k (1%)
- R21: value 0.1 (0.5W) -> 240k (1%)
- R22: value 10k (1%) -> 1M
- R23: value 220k (1%) -> 220 (1W)
- R28: value 470k -> 220 (1W)
- R29: value 10 -> 3.9K
- R36, R41: value 10 -> 220k
- R38: value 470k -> 470
- R39: value 10 -> 470
- R40: value 220 -> 10k
- R42: value 1M -> 10k
- R44: value 1M -> 220k
- R49: value 10 -> 220 (1W)
- R54: value 100k -> 10k
- R55: value 10k -> 22k
- R56: value 220k (1%) -> 240k (1%)
- R57: value 0.1 (0.5W) -> 47k
- R58: value 47k (1%) -> 220k
- R59, R62: value 220k (1%) -> 10k
- R60: value 10k (1%) -> 15k
- R61: value 470k -> 1k
- R63: value 10 -> 10k
- R7: value 1k -> 10k
- SW1: value RESET MANUAL -> ON/OFF 2
- SW4: value RESET MANUAL -> ON/OFF 1
- renumbered J7 to IN_BAT, J5 to IN_PANEL
Connections:
- net +3.3V: now also D32.2 (A), SENSOR_TEMP.3 (Pin_3); no longer J3.6 (Pin_6), J9.6 (Pin_6)
- net +5V: now also C16.2, C8.1, R57.1, R58.2, R61.1, ACS3.1 (Pin_1), ACS712.1 (Pin_1), U3.4 (R), U3.8 (VCC); no longer C11.2, C17.2
- net ADC V1: now also C10.1, LEFT_ESP1.4 (Pin_4); no longer LEFT_ESP1.2 (Pin_2)
- net ADC V2: now also C11.1, LEFT_ESP1.5 (Pin_5), R20.2, R21.2; no longer LEFT_ESP1.3 (Pin_3), R58.2, R59.2
- net ALARMA SC 1: now also LEFT_ESP1.8 (Pin_8), R1.2; no longer RIGHT_ESP1.6 (Pin_6)
- net ALARMA SC 2: now also LEFT_ESP1.9 (Pin_9), R59.2, R60.2; no longer RIGHT_ESP1.5 (Pin_5)
- net GND: now also C11.2, C13.1, C15.2, C17.2, C8.2, D10.2 (A2), D12.2 (A2), J2.1 (Pin_1), R15.1, R16.2, R17.1, R20.1, R22.2, R29.1, R41.1, R55.1, R63.1, R64.1, ACS6.1 (Pin_1), ACS712.1 (Pin_1), C18.2, C6.2, D15.1 (K), D16.2 (A), D2.2 (A2), D29.2 (A), D33.2 (A), D34.1 (K), D9.2 (A), J4.1 (Pin_1), Q1.3 (E), Q10.3 (E), Q13.3 (E), Q17.3 (E), Q18.3 (E), Q19.3 (E), Q2.3 (E), Q4.3 (E), Q5.3 (E), R80.1, SENSOR_TEMP.1 (Pin_1), U3.1 (GND); no longer C11.1, C12.2, C13.2, C15.1, C17.1, C8.1, R17.2, R20.2, R21.2, R22.1, R28.2, R38.2, R43.2, R54.1, R57.2, R58.1, R61.2
- net ON/OFF 1: now also LEFT_ESP1.7 (Pin_7); no longer RIGHT_ESP1.15 (Pin_15)
- net ON/OFF 2: now also D24.2 (A), LEFT_ESP1.10 (Pin_10); no longer RIGHT_ESP1.10 (Pin_10)
- net PWM: now also LEFT_ESP1.13 (Pin_13); no longer RIGHT_ESP1.9 (Pin_9)
- net RESET MODEM: now also LEFT_ESP1.12 (Pin_12); no longer LEFT_ESP1.6 (Pin_6)
- net VCC: now also R44.1, D17.1 (K), D19.1 (K), D20.1 (K), D21.1 (K), Q3.3 (S); no longer C10.1, R44.2
- net at D4.1 (K): now also R1.1, U2.3 (Q)
- net at C5.2, D10.1 (A1), D7.2 (A)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: now also ACS712.1 (Pin_1); no longer D5.1 (K), Q6.2 (D), R16.2
- net at R50.2, R51.1: now also Q17.1 (C)
- net at J9.1 (Pin_1), R46.1, R47.1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: now also F2.2, R37.2; no longer Q12.2 (D)
- net at R27.1, R33.1: now also Q10.1 (C)
- net at D7.1 (K): now also R16.1; no longer R17.1
- net at R30.1: now also Q8.1 (G), D29.1 (K), D9.1 (K); no longer R29.2
- net at D11.2 (A), D12.1 (A1), DCDC8.1 (Pin_1)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: no longer C12.1
- net at R3.2: now also C7.1, R17.2, U2.6 (THR)
- net at C4.1, R9.1, U1.3: now also Q2.1 (C)
- net at R63.2: now also R62.1, C19.2, D22.2 (A)
- net at R24.1, U1.2, U2.2 (TR): now also C6.1, Q1.1 (C); no longer C8.2
- net at R55.2: now also C17.1, R42.2, U3.6 (THR); no longer R54.2
- net at R23.1: now also Q4.1 (C); no longer R22.2
- net at J1.2 (Pin_2), Q6.3 (S), R14.1: now also D6.1 (K), D8.1 (K)
- net at R12.2, R14.2: now also Q6.1 (G), D6.2 (A), D8.2 (A); no longer R13.2
- net at R11.1, U1.4, U2.7 (DIS): now also R10.1; no longer R10.2, R15.1
- net at Q11.1 (G): now also R37.1, D16.1 (K), D33.1 (K); no longer R36.1
- net at R36.2: now also Q12.1 (G), R28.1, D13.2 (A), D30.2 (A); no longer R37.1
- net at J3.1 (Pin_1), R25.1, R26.1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: now also Q12.3 (S), R36.1, D13.1 (K), D30.1 (K)
- net at R11.2: now also R13.2, R15.2, Q18.2 (B)
- net at R12.1: now also Q18.1 (C)
- net at R45.2: now also R41.2, R43.2, Q4.2 (B)
- net at R52.2, R53.2: now also Q17.2 (B)
- net at D24.1 (K), R64.2: now also SW1.1, C19.1; no longer C16.2, R59.1
- net at D11.1 (K): now also R29.2; no longer R28.1
- net at R34.2, R35.2: now also Q10.2 (B)
- net at IN_PANEL.1 (Pin_1), Q8.2 (D): now also C12.2; no longer D12.2 (A2)
- net at F1.1, IN_PANEL.2 (Pin_2): now also C12.1
- net at R62.2: now also Q19.2 (B)
- net at DCDC2.1 (Pin_1): now also Q12.2 (D)
- net at R7.2: now also Q1.2 (B)
- net LED_BAT: now reaches RIGHT_ESP1.3 (Pin_3)
- net LED_BAT: now also R38.2
- net at R39.1: now also D34.2 (A); no longer Q12.1 (G)
- net at R38.1: now also D15.2 (A)
- net at Q14.1 (G), R49.1: now also D17.2 (A), D19.2 (A)
- net at R13.1: now also D5.1 (K), Q6.2 (D), ACS712.1 (Pin_1); no longer Q6.1 (G)
- net at R40.2: now also Q13.2 (B), R80.2
- net TEMP: now reaches LEFT_ESP1.11 (Pin_11)
- net TEMP: now also SENSOR_TEMP.2 (Pin_2)
- net CORTE BAT: no longer names the net of RIGHT_ESP1.7 (Pin_7)
- new net: D32.1 (K), J3.6 (Pin_6), J9.6 (Pin_6)
- new net: D20.2 (A), D21.2 (A), Q3.1 (G), R23.2, R44.2
- new net: ACS4.1 (Pin_1), R42.1
- new net: D31.1 (K), R40.1
- new net: ACS5.1 (Pin_1), D22.1 (K), Q3.2 (D), R43.1
- new net: C14.1, Q19.1 (C), R22.1, U3.2 (TR), U4.2
- new net: C18.1, Q5.1 (C), R58.1, U4.3
- new net: Q5.2 (B), R54.2
- new net: R61.2, U4.1
- new net: D23.1 (K), R59.1, U3.3 (Q)
- new net: D23.2 (A), R57.2
- new net: Q2.2 (B), R10.2
- new net: ACS2.1 (Pin_1), C13.2, D2.1 (A1), D3.2 (A), J4.2 (Pin_2), R21.1
- new net: Q13.1 (C), R28.2
- new net: R45.1, R54.1, U3.7 (DIS), U4.4
- new net: C15.1, U3.5 (CV)
- new net: ACS1.1 (Pin_1), R3.1
- new net: D3.1 (K), R18.1
- new net CORTE_INPANEL: D31.2 (A), LEFT_ESP1.6 (Pin_6)
- new net LED_ESTADO: R39.2, RIGHT_ESP1.5 (Pin_5)
Other:
- note added: "3V3"
- note removed: "VCC"
- moved on the sheet: C1, C2, C3, C4, C5, C7, D1, D10, D11, D14, D18, D5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
