File: Testing/Testing Emiliano/PCB_REGULADOR_SOLAR/pcb_regulador_solar_V1.0/pcb_regulador_solar_V1.0.kicad_pcb (KiCad board)
At the start: 2 copper layers, 0 parts

Commit message: Armado PCB
Parts:
- added C1: 100nf, Capacitor_THT:C_Axial_L5.1mm_D3.1mm_P7.50mm_Horizontal, F.Cu at (-76.7, 17.3)
- added C10: 100n, Capacitor_THT:C_Axial_L5.1mm_D3.1mm_P7.50mm_Horizontal, F.Cu at (216.0, 78.7)
- added C11: 100nf, Capacitor_THT:C_Axial_L5.1mm_D3.1mm_P7.50mm_Horizontal, F.Cu at (-66.0, 22.0)
- added C12: 100n, Capacitor_THT:C_Axial_L5.1mm_D3.1mm_P7.50mm_Horizontal, F.Cu at (-66.0, 26.6)
- added C13: 100n, Capacitor_THT:C_Axial_L5.1mm_D3.1mm_P7.50mm_Horizontal, F.Cu at (160.5, 103.2)
- added C14: 100u 25v, Capacitor_THT:C_Radial_D5.0mm_H11.0mm_P2.00mm, F.Cu at (163.1, 127.0)
- added C15: 10nf, Capacitor_THT:C_Axial_L5.1mm_D3.1mm_P7.50mm_Horizontal, F.Cu at (-66.0, 35.9)
- added C16: 100nf, Capacitor_THT:C_Axial_L5.1mm_D3.1mm_P7.50mm_Horizontal, F.Cu at (-66.0, 40.6)
- added C17: 100nf, Capacitor_THT:C_Axial_L5.1mm_D3.1mm_P7.50mm_Horizontal, F.Cu at (-55.4, 17.3)
- added C18: 100nf, Capacitor_THT:C_Axial_L5.1mm_D3.1mm_P7.50mm_Horizontal, F.Cu at (-55.4, 22.0)
- added C19: 10nf, Capacitor_THT:C_Axial_L5.1mm_D3.1mm_P7.50mm_Horizontal, F.Cu at (-55.4, 26.6)
- added C2: 10nf, Capacitor_THT:C_Axial_L5.1mm_D3.1mm_P7.50mm_Horizontal, F.Cu at (-76.7, 22.0)
- added C20: 10nf, Capacitor_THT:C_Axial_L5.1mm_D3.1mm_P7.50mm_Horizontal, F.Cu at (-55.4, 31.3)
- added C21: 100nf, Capacitor_THT:C_Axial_L5.1mm_D3.1mm_P7.50mm_Horizontal, F.Cu at (-55.4, 35.9)
- added C22: 22u 25v, Capacitor_THT:C_Radial_D5.0mm_H11.0mm_P2.00mm, F.Cu at (211.4, 111.8)
- added C23: 47u 16v, Capacitor_THT:C_Radial_D5.0mm_H11.0mm_P2.00mm, F.Cu at (211.4, 119.4)
- added C3: 47u 16v, Capacitor_THT:C_Radial_D5.0mm_H11.0mm_P2.00mm, F.Cu at (204.3, 119.4)
- added C4: 22u 25v, Capacitor_THT:C_Radial_D5.0mm_H11.0mm_P2.00mm, F.Cu at (204.3, 111.8)
- added C5: 100nf, Capacitor_THT:C_Axial_L5.1mm_D3.1mm_P7.50mm_Horizontal, F.Cu at (223.6, 140.1)
- added C6: 10nf, Capacitor_THT:C_Axial_L5.1mm_D3.1mm_P7.50mm_Horizontal, F.Cu at (223.6, 144.8)
- added C7: 10nf, Capacitor_THT:C_Axial_L5.1mm_D3.1mm_P7.50mm_Horizontal, F.Cu at (-76.7, 35.9)
- added C8: 100nf, Capacitor_THT:C_Axial_L5.1mm_D3.1mm_P7.50mm_Horizontal, F.Cu at (-76.7, 40.6)
- added C9: 1000u 25v, Capacitor_THT:C_Radial_D10.0mm_H20.0mm_P5.00mm, F.Cu at (198.1, 73.7)
- added D1: 1N5819, Diode_THT:D_DO-41_SOD81_P10.16mm_Horizontal, F.Cu at (-89.3, 69.4)
- added D10: 1.5KE18, Diode_THT:D_DO-201AE_P15.24mm_Horizontal, F.Cu at (190.5, 139.7)
- added D11: LED VERDE, LED_THT:LED_D3.0mm_IRBlack, F.Cu at (124.5, 149.9)
- added D12: 1.5KE30A, Diode_THT:D_DO-201AE_P15.24mm_Horizontal, F.Cu at (129.5, 129.5)
- added D13: 18v, Diode_THT:D_DO-35_SOD27_P7.62mm_Horizontal, F.Cu at (160.0, 109.2)
- added D14: 1N5819, Diode_THT:D_DO-41_SOD81_P10.16mm_Horizontal, F.Cu at (-89.3, 82.1)
- added D15: 18v, Diode_THT:D_DO-35_SOD27_P7.62mm_Horizontal, F.Cu at (160.0, 113.3)
- added D16: 18v, Diode_THT:D_DO-35_SOD27_P7.62mm_Horizontal, F.Cu at (160.0, 116.8)
- added D17: LED VERDE, LED_THT:LED_D3.0mm_IRBlack, F.Cu at (149.9, 149.9)
- added D18: 1N5819, Diode_THT:D_DO-41_SOD81_P10.16mm_Horizontal, F.Cu at (-89.3, 86.4)
- added D19: 1N5819, Diode_THT:D_DO-41_SOD81_P10.16mm_Horizontal, F.Cu at (-89.3, 90.6)
- added D2: 1N5819, Diode_THT:D_DO-41_SOD81_P10.16mm_Horizontal, F.Cu at (-89.3, 73.6)
- added D20: 1.5KE18, Diode_THT:D_DO-201AE_P15.24mm_Horizontal, F.Cu at (180.3, 116.8)
- added D21: 3.3, Diode_THT:D_DO-35_SOD27_P7.62mm_Horizontal, F.Cu at (-66.5, 90.3)
- added D22: LED VERDE, LED_THT:LED_D3.0mm_IRBlack, F.Cu at (215.9, 152.4)
- added D23: 18v, Diode_THT:D_DO-35_SOD27_P7.62mm_Horizontal, F.Cu at (-66.5, 93.9)
- added D24: 1N5819, Diode_THT:D_DO-41_SOD81_P10.16mm_Horizontal, F.Cu at (-89.3, 94.9)
- added D25: 1N5819, Diode_THT:D_DO-41_SOD81_P10.16mm_Horizontal, F.Cu at (-89.3, 99.1)
- added D26: 3.3, Diode_THT:D_DO-35_SOD27_P7.62mm_Horizontal, F.Cu at (-66.5, 97.4)
- added D27: LED ROJO, LED_THT:LED_D3.0mm_IRBlack, F.Cu at (215.9, 144.8)
- added D28: 1N5819, Diode_THT:D_DO-41_SOD81_P10.16mm_Horizontal, F.Cu at (-89.3, 103.4)
- added D3: 3.3, Diode_THT:D_DO-35_SOD27_P7.62mm_Horizontal, F.Cu at (-66.5, 69.0)
- added D4: LED ROJO, LED_THT:LED_D3.0mm_IRBlack, F.Cu at (182.9, 144.8)
- added D5: 1N5819, Diode_THT:D_DO-41_SOD81_P10.16mm_Horizontal, F.Cu at (-89.3, 77.9)
- added D6: 18v, Diode_THT:D_DO-35_SOD27_P7.62mm_Horizontal, F.Cu at (196.8, 128.5)
- added D7: LED VERDE, LED_THT:LED_D3.0mm_IRBlack, F.Cu at (182.9, 152.4)
- added D8: 3.3, Diode_THT:D_DO-35_SOD27_P7.62mm_Horizontal, F.Cu at (196.8, 132.1)
- added D9: 1N5822, Diode_THT:D_DO-201AD_P15.24mm_Horizontal, F.Cu at (190.5, 116.8)
- added DCDC1: IN-, Connector_PinHeader_2.54mm:PinHeader_1x01_P2.54mm_Vertical, F.Cu at (121.9, 66.0)
- added DCDC2: OUT+, Connector_PinHeader_2.54mm:PinHeader_1x01_P2.54mm_Vertical, F.Cu at (165.1, 45.7)
- added DCDC3: OUT-, Connector_PinHeader_2.54mm:PinHeader_1x01_P2.54mm_Vertical, F.Cu at (165.1, 66.0)
- added DCDC4: IN+, Connector_PinHeader_2.54mm:PinHeader_1x01_P2.54mm_Vertical, F.Cu at (193.0, 43.2)
- added DCDC5: IN-, Connector_PinHeader_2.54mm:PinHeader_1x01_P2.54mm_Vertical, F.Cu at (193.0, 63.5)
- added DCDC6: OUT+, Connector_PinHeader_2.54mm:PinHeader_1x01_P2.54mm_Vertical, F.Cu at (236.2, 43.2)
- added DCDC7: OUT-, Connector_PinHeader_2.54mm:PinHeader_1x01_P2.54mm_Vertical, F.Cu at (236.2, 63.5)
- added DCDC8: IN+, Connector_PinHeader_2.54mm:PinHeader_1x01_P2.54mm_Vertical, F.Cu at (121.9, 45.7)
- added F1: Fuse 3A, Fuse:Fuseholder_Clip-5x20mm_Bel_FC-203-22_Lateral_P17.80x5.00mm_D1.17mm_Horizontal, F.Cu at (144.8, 139.6)
- added F2: Fuse 3A, Fuse:Fuseholder_Clip-5x20mm_Bel_FC-203-22_Lateral_P17.80x5.00mm_D1.17mm_Horizontal, F.Cu at (151.1, 134.7)
- added J1: Conn_01x03_Pin, Connector_PinHeader_2.54mm:PinHeader_1x03_P2.54mm_Vertical, F.Cu at (-76.0, 45.2)
- added J10: Conn_01x03_Pin, Connector_PinHeader_2.54mm:PinHeader_1x03_P2.54mm_Vertical, F.Cu at (-71.3, 45.2)
- added J2: Screw_Terminal_01x02, TerminalBlock:TerminalBlock_bornier-2_P5.08mm, F.Cu at (190.5, 152.4)
- added J3: INA219, Connector_PinSocket_2.54mm:PinSocket_1x06_P2.54mm_Vertical, F.Cu at (213.4, 73.7)
- added J4: Conn_01x02_Pin, Connector_PinHeader_2.54mm:PinHeader_1x02_P2.54mm_Vertical, F.Cu at (-66.7, 45.2)
- added J5: Screw_Terminal_01x02, TerminalBlock:TerminalBlock_bornier-2_P5.08mm, F.Cu at (132.1, 149.9)
- added J6: USB_A, Connector_USB:USB_A_Wuerth_614004134726_Horizontal, F.Cu at (125.2, 37.9)
- added J7: Screw_Terminal_01x02, TerminalBlock:TerminalBlock_bornier-2_P5.08mm, F.Cu at (157.5, 149.9)
- added J8: Screw_Terminal_01x02, TerminalBlock:TerminalBlock_bornier-2_P5.08mm, F.Cu at (223.5, 152.4)
- added J9: INA219, Connector_PinSocket_2.54mm:PinSocket_1x06_P2.54mm_Vertical, F.Cu at (134.6, 76.2)
- added LEFT_ESP1: L ESP, Connector_PinSocket_2.54mm:PinSocket_1x15_P2.54mm_Vertical, F.Cu at (172.7, 86.3)
- added Q1: BC557, Package_TO_SOT_THT:TO-92_Inline, F.Cu at (221.9, 111.5)
- added Q10: 2N3904, Package_TO_SOT_THT:TO-92_Inline, F.Cu at (218.4, 38.1)
- added Q11: IRLIZ44N, Package_TO_SOT_THT:TO-220F-3_Vertical, F.Cu at (119.4, 109.2)
- added Q12: IRF4905, Package_TO_SOT_THT:TO-220-3_Vertical, F.Cu at (119.4, 96.5)
- added Q13: 2N7000, Package_TO_SOT_THT:TO-92_Inline, F.Cu at (149.9, 129.5)
- added Q14: IRF4905, Package_TO_SOT_THT:TO-220-3_Vertical, F.Cu at (119.4, 134.6)
- added Q15: BC337, Package_TO_SOT_THT:TO-92_Inline, F.Cu at (149.9, 121.9)
- added Q16: BC327, Package_TO_SOT_THT:TO-92_Inline, F.Cu at (142.2, 121.9)
- added Q17: 2N3904, Package_TO_SOT_THT:TO-92_Inline, F.Cu at (134.6, 121.9)
- added Q18: 2N3904, Package_TO_SOT_THT:TO-92_Inline, F.Cu at (127.0, 121.9)
- added Q19: IRF4905, Package_TO_SOT_THT:TO-220-3_Vertical, F.Cu at (236.2, 124.5)
- added Q2: BC557, Package_TO_SOT_THT:TO-92_Inline, F.Cu at (222.2, 116.8)
- added Q20: 2N3904, Package_TO_SOT_THT:TO-92_Inline, F.Cu at (229.9, 111.8)
- added Q21: 2N3904, Package_TO_SOT_THT:TO-92_Inline, F.Cu at (230.2, 117.1)
- added Q22: 2N3904, Package_TO_SOT_THT:TO-92_Inline, F.Cu at (230.2, 122.9)
- added Q23: BC557, Package_TO_SOT_THT:TO-92_Inline, F.Cu at (230.2, 128.7)
- added Q24: BC557, Package_TO_SOT_THT:TO-92_Inline, F.Cu at (230.2, 134.5)
- added Q3: 2N3904, Package_TO_SOT_THT:TO-92_Inline, F.Cu at (222.2, 122.6)
- added Q4: 2N3904, Package_TO_SOT_THT:TO-92_Inline, F.Cu at (222.2, 128.4)
- added Q5: 2N3904, Package_TO_SOT_THT:TO-92_Inline, F.Cu at (222.2, 134.2)
- added Q6: IRF4905, Package_TO_SOT_THT:TO-220-3_Vertical, F.Cu at (236.2, 137.2)
- added Q7: IRF4905, Package_TO_SOT_THT:TO-220-3_Vertical, F.Cu at (233.7, 30.5)
- added Q8: IRLIZ44N, Package_TO_SOT_THT:TO-220F-3_Vertical, F.Cu at (119.4, 121.9)
- added Q9: BC557, Package_TO_SOT_THT:TO-92_Inline, F.Cu at (224.8, 38.1)
- added R1: 10k, Resistor_THT:R_Axial_DIN0207_L6.3mm_D2.5mm_P2.54mm_Vertical, F.Cu at (-125.4, 17.0)
- added R10: 10k, Resistor_THT:R_Axial_DIN0207_L6.3mm_D2.5mm_P2.54mm_Vertical, F.Cu at (-125.4, 53.5)
- added R11: 10k, Resistor_THT:R_Axial_DIN0207_L6.3mm_D2.5mm_P2.54mm_Vertical, F.Cu at (-119.2, 17.0)
- added R12: 220, Resistor_THT:R_Axial_DIN0207_L6.3mm_D2.5mm_P2.54mm_Vertical, F.Cu at (-119.2, 21.1)
- added R13: 10, Resistor_THT:R_Axial_DIN0207_L6.3mm_D2.5mm_P2.54mm_Vertical, F.Cu at (236.2, 111.8)
- added R14: 220k, Resistor_THT:R_Axial_DIN0207_L6.3mm_D2.5mm_P2.54mm_Vertical, F.Cu at (-119.2, 29.2)
- added R15: 220k, Resistor_THT:R_Axial_DIN0207_L6.3mm_D2.5mm_P2.54mm_Vertical, F.Cu at (-119.2, 33.2)
- added R16: 10k, Resistor_THT:R_Axial_DIN0207_L6.3mm_D2.5mm_P2.54mm_Vertical, F.Cu at (236.2, 116.8)
- added R17: 470k, Resistor_THT:R_Axial_DIN0207_L6.3mm_D2.5mm_P2.54mm_Vertical, F.Cu at (-119.2, 41.3)
- added R18: 0.1 (0.5W), Resistor_THT:R_Axial_DIN0207_L6.3mm_D2.5mm_P2.54mm_Vertical, F.Cu at (-119.2, 45.4)
- added R19: 47k (1%), Resistor_THT:R_Axial_DIN0207_L6.3mm_D2.5mm_P2.54mm_Vertical, F.Cu at (228.6, 94.0)
- added R2: 100k, Resistor_THT:R_Axial_DIN0207_L6.3mm_D2.5mm_P2.54mm_Vertical, F.Cu at (-125.4, 21.1)
- added R20: 0.1 (0.5W), Resistor_THT:R_Axial_DIN0207_L6.3mm_D2.5mm_P2.54mm_Vertical, F.Cu at (228.6, 98.0)
- added R21: 0.1 (0.5W), Resistor_THT:R_Axial_DIN0207_L6.3mm_D2.5mm_P2.54mm_Vertical, F.Cu at (235.5, 96.6)
- added R22: 10k (1%), Resistor_THT:R_Axial_DIN0207_L6.3mm_D2.5mm_P2.54mm_Vertical, F.Cu at (235.5, 100.7)
- added R23: 220k (1%), Resistor_THT:R_Axial_DIN0207_L6.3mm_D2.5mm_P2.54mm_Vertical, F.Cu at (235.5, 104.7)
- added R24: 1M, Resistor_THT:R_Axial_DIN0207_L6.3mm_D2.5mm_P2.54mm_Vertical, F.Cu at (-113.1, 29.2)
- added R25: 0,1 (2w), Resistor_THT:R_Axial_DIN0207_L6.3mm_D2.5mm_P2.54mm_Vertical, F.Cu at (233.7, 73.7)
- added R26: 0,1 (2w), Resistor_THT:R_Axial_DIN0207_L6.3mm_D2.5mm_P2.54mm_Vertical, F.Cu at (233.7, 81.3)
- added R27: 10k, Resistor_THT:R_Axial_DIN0207_L6.3mm_D2.5mm_P2.54mm_Vertical, F.Cu at (-113.1, 41.3)
- added R28: 470k, Resistor_THT:R_Axial_DIN0207_L6.3mm_D2.5mm_P2.54mm_Vertical, F.Cu at (-113.1, 45.4)
- added R29: 10, Resistor_THT:R_Axial_DIN0207_L6.3mm_D2.5mm_P2.54mm_Vertical, F.Cu at (149.9, 83.8)
- added R3: 10k, Resistor_THT:R_Axial_DIN0207_L6.3mm_D2.5mm_P2.54mm_Vertical, F.Cu at (-125.4, 25.1)
- added R30: 220, Resistor_THT:R_Axial_DIN0207_L6.3mm_D2.5mm_P2.54mm_Vertical, F.Cu at (157.5, 86.4)
- added R31: 0,1 (2w), Resistor_THT:R_Axial_DIN0207_L6.3mm_D2.5mm_P2.54mm_Vertical, F.Cu at (233.7, 88.9)
- added R32: 10k, Resistor_THT:R_Axial_DIN0207_L6.3mm_D2.5mm_P2.54mm_Vertical, F.Cu at (-107.0, 21.1)
- added R33: 10k, Resistor_THT:R_Axial_DIN0207_L6.3mm_D2.5mm_P2.54mm_Vertical, F.Cu at (-107.0, 25.1)
- added R34: 10k, Resistor_THT:R_Axial_DIN0207_L6.3mm_D2.5mm_P2.54mm_Vertical, F.Cu at (-107.0, 29.2)
- added R35: 100k, Resistor_THT:R_Axial_DIN0207_L6.3mm_D2.5mm_P2.54mm_Vertical, F.Cu at (-107.0, 33.2)
- added R36: 10, Resistor_THT:R_Axial_DIN0207_L6.3mm_D2.5mm_P2.54mm_Vertical, F.Cu at (149.9, 102.6)
- added R37: 220, Resistor_THT:R_Axial_DIN0207_L6.3mm_D2.5mm_P2.54mm_Vertical, F.Cu at (149.9, 106.7)
- added R38: 470k, Resistor_THT:R_Axial_DIN0207_L6.3mm_D2.5mm_P2.54mm_Vertical, F.Cu at (-107.0, 45.4)
- added R39: 10, Resistor_THT:R_Axial_DIN0207_L6.3mm_D2.5mm_P2.54mm_Vertical, F.Cu at (149.9, 114.8)
- added R4: 47k, Resistor_THT:R_Axial_DIN0207_L6.3mm_D2.5mm_P2.54mm_Vertical, F.Cu at (-125.4, 29.2)
- added R40: 220, Resistor_THT:R_Axial_DIN0207_L6.3mm_D2.5mm_P2.54mm_Vertical, F.Cu at (157.5, 96.5)
- added R41: 10, Resistor_THT:R_Axial_DIN0207_L6.3mm_D2.5mm_P2.54mm_Vertical, F.Cu at (-100.8, 17.0)
- added R42: 1M, Resistor_THT:R_Axial_DIN0207_L6.3mm_D2.5mm_P2.54mm_Vertical, F.Cu at (149.9, 96.5)
- added R43: 1M, Resistor_THT:R_Axial_DIN0207_L6.3mm_D2.5mm_P2.54mm_Vertical, F.Cu at (-100.8, 25.1)
- added R44: 1M, Resistor_THT:R_Axial_DIN0207_L6.3mm_D2.5mm_P2.54mm_Vertical, F.Cu at (-100.8, 29.2)
- added R45: 10k, Resistor_THT:R_Axial_DIN0207_L6.3mm_D2.5mm_P2.54mm_Vertical, F.Cu at (-100.8, 33.2)
- added R46: 0,1 (2w), Resistor_THT:R_Axial_DIN0207_L6.3mm_D2.5mm_P2.54mm_Vertical, F.Cu at (121.9, 77.2)
- added R47: 0,1 (2w), Resistor_THT:R_Axial_DIN0207_L6.3mm_D2.5mm_P2.54mm_Vertical, F.Cu at (121.9, 81.3)
- added R48: 0,1 (2w), Resistor_THT:R_Axial_DIN0207_L6.3mm_D2.5mm_P2.54mm_Vertical, F.Cu at (121.9, 85.3)
- added R49: 10, Resistor_THT:R_Axial_DIN0207_L6.3mm_D2.5mm_P2.54mm_Vertical, F.Cu at (-100.8, 49.4)
- added R5: 10k, Resistor_THT:R_Axial_DIN0207_L6.3mm_D2.5mm_P2.54mm_Vertical, F.Cu at (-125.4, 33.2)
- added R50: 3.9K, Resistor_THT:R_Axial_DIN0207_L6.3mm_D2.5mm_P2.54mm_Vertical, F.Cu at (-100.8, 53.5)
- added R51: 10k, Resistor_THT:R_Axial_DIN0207_L6.3mm_D2.5mm_P2.54mm_Vertical, F.Cu at (-94.7, 17.0)
- added R52: 100k, Resistor_THT:R_Axial_DIN0207_L6.3mm_D2.5mm_P2.54mm_Vertical, F.Cu at (-94.7, 21.1)
- added R53: 10k, Resistor_THT:R_Axial_DIN0207_L6.3mm_D2.5mm_P2.54mm_Vertical, F.Cu at (-94.7, 25.1)
- added R54: 100k, Resistor_THT:R_Axial_DIN0207_L6.3mm_D2.5mm_P2.54mm_Vertical, F.Cu at (-94.7, 29.2)
- added R55: 10k, Resistor_THT:R_Axial_DIN0207_L6.3mm_D2.5mm_P2.54mm_Vertical, F.Cu at (-94.7, 33.2)
- added R56: 220k (1%), Resistor_THT:R_Axial_DIN0207_L6.3mm_D2.5mm_P2.54mm_Vertical, F.Cu at (226.1, 83.8)
- added R57: 0.1 (0.5W), Resistor_THT:R_Axial_DIN0207_L6.3mm_D2.5mm_P2.54mm_Vertical, F.Cu at (-94.7, 41.3)
- added R58: 47k (1%), Resistor_THT:R_Axial_DIN0207_L6.3mm_D2.5mm_P2.54mm_Vertical, F.Cu at (-94.7, 45.4)
- added R59: 220k (1%), Resistor_THT:R_Axial_DIN0207_L6.3mm_D2.5mm_P2.54mm_Vertical, F.Cu at (-94.7, 49.4)
- added R6: 10k, Resistor_THT:R_Axial_DIN0207_L6.3mm_D2.5mm_P2.54mm_Vertical, F.Cu at (-125.4, 37.3)
- added R60: 10k (1%), Resistor_THT:R_Axial_DIN0207_L6.3mm_D2.5mm_P2.54mm_Vertical, F.Cu at (-94.7, 53.5)
- added R61: 470k, Resistor_THT:R_Axial_DIN0207_L6.3mm_D2.5mm_P2.54mm_Vertical, F.Cu at (-88.5, 17.0)
- added R62: 220k (1%), Resistor_THT:R_Axial_DIN0207_L6.3mm_D2.5mm_P2.54mm_Vertical, F.Cu at (-88.5, 21.1)
- added R63: 10, Resistor_THT:R_Axial_DIN0207_L6.3mm_D2.5mm_P2.54mm_Vertical, F.Cu at (-88.5, 25.1)
- added R64: 10k, Resistor_THT:R_Axial_DIN0207_L6.3mm_D2.5mm_P2.54mm_Vertical, F.Cu at (-88.5, 29.2)
- added R65: 220, Resistor_THT:R_Axial_DIN0207_L6.3mm_D2.5mm_P2.54mm_Vertical, F.Cu at (-88.5, 33.2)
- added R66: 220k, Resistor_THT:R_Axial_DIN0207_L6.3mm_D2.5mm_P2.54mm_Vertical, F.Cu at (-88.5, 37.3)
- added R67: 1M, Resistor_THT:R_Axial_DIN0207_L6.3mm_D2.5mm_P2.54mm_Vertical, F.Cu at (-88.5, 41.3)
- added R68: 10k, Resistor_THT:R_Axial_DIN0207_L6.3mm_D2.5mm_P2.54mm_Vertical, F.Cu at (-88.5, 45.4)
- added R69: 220k, Resistor_THT:R_Axial_DIN0207_L6.3mm_D2.5mm_P2.54mm_Vertical, F.Cu at (-88.5, 49.4)
- added R7: 1k, Resistor_THT:R_Axial_DIN0207_L6.3mm_D2.5mm_P2.54mm_Vertical, F.Cu at (-125.4, 41.3)
- added R70: 10k, Resistor_THT:R_Axial_DIN0207_L6.3mm_D2.5mm_P2.54mm_Vertical, F.Cu at (-88.5, 53.5)
- added R71: 220k, Resistor_THT:R_Axial_DIN0207_L6.3mm_D2.5mm_P2.54mm_Vertical, F.Cu at (-82.4, 17.0)
- added R72: 1k, Resistor_THT:R_Axial_DIN0207_L6.3mm_D2.5mm_P2.54mm_Vertical, F.Cu at (-82.4, 21.1)
- added R73: 1k, Resistor_THT:R_Axial_DIN0207_L6.3mm_D2.5mm_P2.54mm_Vertical, F.Cu at (-82.4, 25.1)
- added R74: 10k, Resistor_THT:R_Axial_DIN0207_L6.3mm_D2.5mm_P2.54mm_Vertical, F.Cu at (-82.4, 29.2)
- added R75: 10k, Resistor_THT:R_Axial_DIN0207_L6.3mm_D2.5mm_P2.54mm_Vertical, F.Cu at (-82.4, 33.2)
- added R76: 10k, Resistor_THT:R_Axial_DIN0207_L6.3mm_D2.5mm_P2.54mm_Vertical, F.Cu at (-82.4, 37.3)
- added R77: 47k, Resistor_THT:R_Axial_DIN0207_L6.3mm_D2.5mm_P2.54mm_Vertical, F.Cu at (-82.4, 41.3)
- added R78: 10k, Resistor_THT:R_Axial_DIN0207_L6.3mm_D2.5mm_P2.54mm_Vertical, F.Cu at (-82.4, 45.4)
- added R79: 100k, Resistor_THT:R_Axial_DIN0207_L6.3mm_D2.5mm_P2.54mm_Vertical, F.Cu at (-82.4, 49.4)
- added R8: 1k, Resistor_THT:R_Axial_DIN0207_L6.3mm_D2.5mm_P2.54mm_Vertical, F.Cu at (-125.4, 45.4)
- added R9: 220k, Resistor_THT:R_Axial_DIN0207_L6.3mm_D2.5mm_P2.54mm_Vertical, F.Cu at (-125.4, 49.4)
- added RIGHT_ESP1: R ESP, Connector_PinSocket_2.54mm:PinSocket_1x15_P2.54mm_Vertical, F.Cu at (198.1, 121.9)
- added SW1: RESET MANUAL, Button_Switch_SMD:SW_SPST_CK_RS282G05A3, F.Cu at (236.2, 151.2)
- added SW2: RESET MANUAL, Button_Switch_SMD:SW_SPST_CK_RS282G05A3, F.Cu at (167.6, 148.7)
- added SW4: RESET MANUAL, Button_Switch_SMD:SW_SPST_CK_RS282G05A3, F.Cu at (203.2, 149.9)
- added U1: PC817, Package_DIP:DIP-4_W7.62mm, F.Cu at (203.2, 92.0)
- added U2: NE555P, Package_DIP:DIP-8_W7.62mm, F.Cu at (200.7, 48.3)
- added U3: PC817, Package_DIP:DIP-4_W7.62mm, F.Cu at (203.2, 98.7)
- added U4: LM358, Package_DIP:DIP-8_W7.62mm, F.Cu at (209.6, 127.0)
- added U5: LM358, Package_DIP:DIP-8_W7.62mm, F.Cu at (136.5, 50.8)
- added U6: PC817, Package_DIP:DIP-4_W7.62mm, F.Cu at (215.9, 92.4)
- added U7: NE555P, Package_DIP:DIP-8_W7.62mm, F.Cu at (147.3, 50.8)
- added U8: PC817, Package_DIP:DIP-4_W7.62mm, F.Cu at (215.9, 99.1)
