File: Testing/Testing Emiliano/PCB_REGULADOR_SOLAR/pcb_módulo_control/pcb_módulo_control.kicad_sch (KiCad schematic)
At the start: 22 parts, among them J6 USB_A, Q10 BC546, Q7 IRF4905, Q9 BC557

Commit message: cambios pcb
Parts:
- removed DCDC4: IN+, Connector_PinHeader_2.54mm:PinHeader_1x01_P2.54mm_Vertical, symbol Connector:Conn_01x01_Pin
- removed DCDC5: IN-, Connector_PinHeader_2.54mm:PinHeader_1x01_P2.54mm_Vertical, symbol Connector:Conn_01x01_Pin
- removed DCDC6: OUT+, Connector_PinHeader_2.54mm:PinHeader_1x01_P2.54mm_Vertical, symbol Connector:Conn_01x01_Pin
- removed DCDC7: OUT-, Connector_PinHeader_2.54mm:PinHeader_1x01_P2.54mm_Vertical, symbol Connector:Conn_01x01_Pin
- added D15: LED VERDE, LED_THT:LED_D3.0mm_IRBlack, symbol Device:LED
- added J9: CONT_OUT2, Connector_PinSocket_2.54mm:PinSocket_1x06_P2.54mm_Vertical, symbol Connector:Conn_01x06_Pin
- added J9: CONT_OUT1, Connector_PinSocket_2.54mm:PinSocket_1x06_P2.54mm_Vertical, symbol Connector:Conn_01x06_Pin
- added R38: 470, Resistor_THT:R_Axial_DIN0207_L6.3mm_D2.5mm_P2.54mm_Vertical, symbol Device:R
- SENSOR_TEMP: value Conn_01x03_Pin -> SENSOR_TEMP1
Connections:
- net GND: now also D15.1 (K)
- net LED_BAT: now also R38.2
- net ON/OFF 1: now also J9.3 (Pin_3)
- net ON/OFF 2: now also J9.3 (Pin_3)
- net ADC V1 renamed ESTADO_OUT1
- net ESTADO_OUT1: now also J9.4 (Pin_4)
- net ADC V2 renamed ESTADO_OUT2
- net ESTADO_OUT2: now also J9.4 (Pin_4)
- net ALARMA SC 1 renamed PROTEC_OUT1
- net PROTEC_OUT1: now also J9.5 (Pin_5)
- net ALARMA SC 2 renamed PROTEC_OUT2
- net PROTEC_OUT2: now also J9.5 (Pin_5)
- new net: D15.2 (A), R38.1
Other:
- note added: "+5V"
- note added: "EST"
- note added: "GND"
- note added: "ON/OFF"
- note added: "PROT"
- moved on the sheet: D34, R39, SENSOR_TEMP
