File: Testing/Testing Emiliano/PCB_REGULADOR_SOLAR/pcb_módulo_energía/pcm_módulo _energía.kicad_sch (KiCad schematic)
At the start: 57 parts, among them J3 INA219, J9 INA219, Q11 IRFZ44N, Q12 IRF4905, Q13 BC546, Q14 IRF4905, Q15 BC337, Q16 BC327, Q17 BC546, Q8 IRFZ44N

Commit message: cambios pcb
Parts:
- removed D15: LED VERDE, LED_THT:LED_D3.0mm_IRBlack, symbol Device:LED
- removed R38: 470, Resistor_THT:R_Axial_DIN0207_L6.3mm_D2.5mm_P2.54mm_Vertical, symbol Device:R
Changed lines of the file:
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@@
-    (stroke (width 0) (type default))
-  )
-  (wire (pts (xy 36.83 110.49) (xy 36.83 105.41))
     (stroke (width 0) (type default))
   )
@@
     (stroke (width 0) (type default))
   )
-  (wire (pts (xy 36.83 127) (xy 36.83 130.81))
-    (stroke (width 0) (type default))
-  )
   (wire (pts (xy 57.15 88.9) (xy 63.5 88.9))
     (stroke (width 0) (type default))
@@
     (stroke (width 0) (type default))
   )
-  (wire (pts (xy 36.83 119.38) (xy 36.83 118.11))
-    (stroke (width 0) (type default))
-  )
   (wire (pts (xy 123.19 128.27) (xy 123.19 134.62))
     (stroke (width 0) (type default))
@@
   )
   (wire (pts (xy 127 160.02) (xy 130.81 160.02))
-    (stroke (width 0) (type default))
-  )
-  (wire (pts (xy 36.83 130.81) (xy 44.45 130.81))
     (stroke (width 0) (type default))
   )
@@
     )
   )
-  (global_label "LED_BAT" (shape input) (at 44.45 130.81 0) (fields_autoplaced)
-    (effects (font (size 1.27 1.27)) (justify left))
-    (property "Intersheetrefs" "${INTERSHEET_REFS}" (at 54.5219 130.81 0)
-      (effects (font (size 1.27 1.27)) (justify left) hide)
-    )
-  )
   (global_label "PWM" (shape input) (at 153.67 149.86 0) (fields_autoplaced)
     (effects (font (size 1.27 1.27)) (justify left))
@@
     )
   )
-  (symbol (lib_id "Device:LED") (at 36.83 114.3 90) (mirror x) (unit 1)
-    (in_bom yes) (on_board yes) (dnp no) (fields_autoplaced)
-    (property "Reference" "D15" (at 40.64 113.9825 90)
-      (effects (font (size 1.27 1.27)) (justify right))
-    )
-    (property "Value" "LED VERDE" (at 40.64 111.4425 90)
-      (effects (font (size 1.27 1.27)) (justify right))
-    )
-    (property "Footprint" "LED_THT:LED_D3.0mm_IRBlack" (at 36.83 114.3 0)
-      (effects (font (size 1.27 1.27)) hide)
-    )
-    (property "Datasheet" "~" (at 36.83 114.3 0)
-      (effects (font (size 1.27 1.27)) hide)
-    )
-    (pin "1")
-    (pin "2")
-    (instances
-      (project "pcb_regulador_solar_V1.0"
-        (path "/152259b8-5bed-4e4f-ac86-e21bf27de3b9"
-          (reference "D15") (unit 1)
-        )
-      )
-      (project "pcm_módulo _energía"
-        (path "/e3e9a0e8-d08b-4640-a2d4-ba40abed7cc8"
-          (reference "D1") (unit 1)
-        )
-      )
-    )
-  )
   (symbol (lib_id "Device:R") (at 175.26 71.12 270) (unit 1)
     (in_bom yes) (on_board yes) (dnp no) (fields_autoplaced)
@@
     )
   )
-  (symbol (lib_id "power:GND") (at 36.83 105.41 0) (mirror x) (unit 1)
-    (in_bom yes) (on_board yes) (dnp no) (fields_autoplaced)
-    (property "Reference" "#PWR035" (at 36.83 99.06 0)
-      (effects (font (size 1.27 1.27)) hide)
-    )
-    (property "Value" "GND" (at 36.83 100.33 0)
-      (effects (font (size 1.27 1.27)))
-    )
-    (property "Footprint" "" (at 36.83 105.41 0)
-      (effects (font (size 1.27 1.27)) hide)
-    )
-    (property "Datasheet" "" (at 36.83 105.41 0)
-      (effects (font (size 1.27 1.27)) hide)
-    )
-    (pin "1")
-    (instances
-      (project "pcb_regulador_solar_V1.0"
-        (path "/152259b8-5bed-4e4f-ac86-e21bf27de3b9"
-          (reference "#PWR035") (unit 1)
-        )
-      )
-      (project "pcm_módulo _energía"
-        (path "/e3e9a0e8-d08b-4640-a2d4-ba40abed7cc8"
-          (reference "#PWR01") (unit 1)
-        )
-      )
-    )
-  )
   (symbol (lib_id "Diode:1N47xxA") (at 87.63 129.54 90) (unit 1)
     (in_bom yes) (on_board yes) (dnp no) (fields_autoplaced)
@@
         )
       )
-    )
-  )
-  (symbol (lib_id "Device:R") (at 36.83 123.19 0) (unit 1)
-    (in_bom yes) (on_board yes) (dnp no) (fields_autoplaced)
-    (property "Reference" "R38" (at 39.37 121.92 0)
-      (effects (font (size 1.27 1.27)) (justify left))
-    )
-    (property "Value" "470" (at 39.37 124.46 0)
-      (effects (font (size 1.27 1.27)) (justify left))
-    )
-    (property "Footprint" "Resistor_THT:R_Axial_DIN0207_L6.3mm_D2.5mm_P2.54mm_Vertical" (at 35.052 123.19 90)
-      (effects (font (size 1.27 1.27)) hide)
-    )
-    (property "Datasheet" "~" (at 36.83 123.19 0)
-      (effects (font (size 1.27 1.27)) hide)
-    )
-    (pin "1")
-    (pin "2")
-    (instances
-      (project "pcb_regulador_solar_V1.0"
-        (path "/152259b8-5bed-4e4f-ac86-e21bf27de3b9"
-          (reference "R38") (unit 1)
-        )
-      )
-      (project "pcm_módulo _energía"
-        (path "/e3e9a0e8-d08b-4640-a2d4-ba40abed7cc8"
-          (reference "R1") (unit 1)
-        )
-      )
