File: Testing/Testing Emiliano/PCB_REGULADOR_SOLAR/pcb_módulo_salida/pcb_módulo_salida.kicad_sch (KiCad schematic)
At the start: 52 parts, among them J2 IN, J2 IN 5V, J2 OUT, J9 CONT, Q1 BC546, Q18 BC546, Q2 BC546, Q6 IRF4905, SW4 ON/OFF 1, U1 PC817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

Commit message: cambios pcb
Parts:
- added J1: selector V salida, Connector_PinHeader_2.54mm:PinHeader_1x03_P2.54mm_Vertical, symbol Connector:Conn_01x03_Pin
- J9: value CONT -> CONTROL
Connections:
- net +5V: now also J9.1 (Pin_1), J1.1 (Pin_1)
- net V+: now also J1.3 (Pin_3); no longer D6.1 (K), D8.1 (K), J9.1 (Pin_1), Q6.3 (S), R14.1
- new net: D6.1 (K), D8.1 (K), J1.2 (Pin_2), Q6.3 (S), R14.1
Other:
- note added: "+5V"
- note added: "GND"
- note removed: "V+"
- note removed: "V-"
- moved on the sheet: J2
