File: Productivo/Tesseract/PCB/Teseracto/Teseracto.kicad_pcb (KiCad board)
At the start: 2 copper layers, 100 x 100 mm, 72 parts, among them J11 LECTOR, J14 jumpers salida, J17 BTN, J3 jumpers salida, J4 IN 12V, J5 FLASH, J6 OUT 1, J7 AUX, J8 PROG, J9 SENS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

Commit message: agregué sim800l
Parts:
- added C5: 1000uF/ 6.3V, Capacitor_SMD:CP_Elec_8x10, F.Cu at (149.5, 54.4)
- added D19: 1N4007 (M7), Diode_SMD:D_MELF, F.Cu at (156.7, 61.5)
- added J10: soporte, Connector_PinHeader_2.54mm:PinHeader_1x05_P2.54mm_Vertical, F.Cu at (115.8, 35.5)
- added J12: SIM800L, Connector_PinHeader_2.54mm:PinHeader_1x05_P2.54mm_Vertical, F.Cu at (98.2, 36.0)
- added J13: PROG, Connector_PinSocket_2.54mm:PinSocket_2x04_P2.54mm_Vertical, F.Cu at (165.5, 61.6)
- added J8: TX_select, Connector_PinHeader_2.54mm:PinHeader_1x03_P2.54mm_Vertical, F.Cu at (162.3, 51.8)
- added Q2: MMBT5551L, Package_TO_SOT_SMD:SOT-23, F.Cu at (155.2, 70.2)
- added R24: 4K7, Diode_SMD:D_MELF, F.Cu at (156.7, 65.8)
- added R25: 10K, Resistor_SMD:R_0805_2012Metric_Pad1.20x1.40mm_HandSolder, F.Cu at (157.7, 53.9)
- added R26: 100K, Resistor_SMD:R_0805_2012Metric_Pad1.20x1.40mm_HandSolder, F.Cu at (157.7, 56.8)
- added R3: 10K, Resistor_SMD:R_0805_2012Metric_Pad1.20x1.40mm_HandSolder, F.Cu at (157.7, 50.9)
- J5: value FLASH -> RX_select
- moved R16 199.7 mm to (90.0, 97.8)
- moved R17 199.7 mm to (90.0, 100.8)
- moved D18 180.6 mm to (82.2, 97.8)
- moved J7 167.3 mm to (96.5, 114.3)
- moved D17 164.1 mm to (84.0, 105.8)
- moved J9 158.9 mm to (76.8, 115.1)
- moved J17 109.6 mm to (70.2, 37.1)
- moved J11 102.3 mm to (35.8, 37.2)
- moved D1 68.5 mm to (211.1, 130.3)
- moved R13 68.5 mm to (222.4, 105.9)
- moved R19 68.5 mm to (227.2, 105.9)
- moved R7 68.5 mm to (217.7, 105.9)
- moved C3 68.5 mm to (193.7, 125.9)
- moved C4 68.5 mm to (192.7, 133.8)
- moved D15 68.5 mm to (194.1, 114.6)
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Connections:
- J5 pad 1: GPIO0 -> TXP
- J5 pad 2: GND -> TX
- J5 pad 3: GND -> TXD
- U2 pad 6: unconnected-(U2-GPIO12-Pad6) -> GPIO12
Other:
- board text added: "SIM800L"

Commit message: actualizacion pcb tesseracto
Parts:
- removed the J8 at (187.3, 99.5)
- added F1: MF-R050, Fuse:Fuse_Bourns_MF-RHT050, F.Cu at (138.2, 52.1)
- added F2: MF-R110, Fuse:Fuse_Bourns_MF-RHT100, F.Cu at (55.4, 116.8)
- added J15: ~, Connector_PinHeader_2.54mm:PinHeader_1x03_P2.54mm_Vertical, F.Cu at (92.2, 89.8)
- added J16: ~, Connector_PinHeader_2.54mm:PinHeader_1x03_P2.54mm_Vertical, F.Cu at (85.8, 89.8)
- added J18: RFW26, Connector_PinSocket_2.54mm:PinSocket_2x04_P2.54mm_Vertical, F.Cu at (230.5, 34.9)
- L1: value 33 uH -> 33 uH/3.5A
- moved R2 195.5 mm to (31.2, 35.0), turned to 90 degrees
- moved SW2 188.6 mm to (36.0, 38.5), turned to 90 degrees
- moved R4 180.2 mm to (43.5, 143.2)
- moved Q1 176.8 mm to (65.2, 72.3), turned to -90 degrees
- moved D11 173.0 mm to (70.0, 45.5), turned to 180 degrees
- moved R14 163.5 mm to (65.2, 68.5), turned to 180 degrees
- moved R9 163.1 mm to (63.5, 57.2)
- moved R13 157.3 mm to (68.8, 72.2), turned to -90 degrees
- moved J14 155.8 mm to (85.5, 95.8)
- moved R10 155.0 mm to (74.5, 50.5), turned to -90 degrees
- moved RV3 152.3 mm to (65.8, 104.8)
- moved R12 151.8 mm to (72.8, 77.8)
- moved Q3 147.8 mm to (94.2, 80.3)
- moved RV4 145.3 mm to (73.8, 104.8)
- moved J3 144.4 mm to (92.2, 96.0)
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Connections:
- net Net-(D6-K) renamed 12V
- D1 pad 1: +5V -> Net-(D1-K)
- D6 pad 2: +12V -> Net-(D6-A)
- D8 pad 1: +5V -> Net-(D8-K)
- J11 pad 6: +12V -> Net-(J11-Pin_6)
- J14 pad 4: +12V -> 12VOUT
- J14 pad 5: +12V -> 12VOUT
- J3 pad 4: +12V -> 12VOUT
- J3 pad 5: +12V -> 12VOUT
- J4 pad 2: +12V -> Net-(D6-A)
- J5 pad 3: TXD -> RXD
- J8 pad 3: RXD -> TXD
- K1 pad 5: +5V -> Net-(D1-K)
- K2 pad 5: +5V -> Net-(D8-K)
- R1 pad 2: +5V -> Net-(D1-K)
- R12 pad 2: +5V -> Net-(D8-K)
Routing:
- net GND: track 67.4 -> 121.6 mm
- net 12VOUT: track 0.00 -> 53.8 mm
- net +5V: track 0.00 -> 50.9 mm
- net 12V: track 23.1 -> 72.0 mm
- net Net-(J14-Pin_2): track 0.00 -> 44.7 mm
- net Net-(D1-K): track 0.00 -> 35.8 mm
- net Net-(J3-Pin_2): track 0.00 -> 29.9 mm
- net Net-(D8-A): track 0.00 -> 26.4 mm
- net Net-(D8-K): track 0.00 -> 23.8 mm
- net Net-(J14-Pin_3): track 0.00 -> 23.7 mm
- net Net-(J3-Pin_3): track 0.00 -> 23.4 mm
- net Net-(D1-A): track 0.00 -> 21.1 mm
- net Net-(D7-K): track 0.00 -> 20.3 mm
- net Net-(J7-Pin_3): track 0.00 -> 18.5 mm
- net Net-(J7-Pin_1): track 0.00 -> 18.3 mm
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Other:
- board size 100 x 100 mm -> 150 x 100 mm
