File: Productivo/RFW26/PCB/RFW26/1 CAPA TESTING/RFW26.kicad_pcb (KiCad board)
At the start: 2 copper layers, 100 x 50 mm, 41 parts, among them J1 IN 12V, J10 OUT, J2 Receptor RF, J3 ESP01, J4 Conn_02x04_Counter_Clockwise, J5 Receptor RF, J6 V-coil1, J9 jumpers salida, K2 SANYOU_SRD_Form_C, Q2 MMBT5551L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

Commit message: correciones RFW26
Parts:
- moved R3 20.9 mm to (73.7, 58.8)
- moved J5 1.91 mm to (58.4, 54.0)
Routing:
- net Net-(J3-Pin_6): track 103.8 -> 6.58 mm, vias 3 -> 0
- net GND: track 341.9 -> 397.7 mm, vias 2 -> 0
- net +3.3V: track 99.3 -> 77.9 mm
- net Net-(J3-Pin_4): track 21.7 -> 9.28 mm, vias 1 -> 0
- net Net-(D1-A): track 47.0 -> 55.7 mm
- net +5V: track 155.1 -> 146.8 mm, vias 1 -> 0
- net Net-(D7-K): track 72.7 -> 79.5 mm
- net D0: track 26.3 -> 31.7 mm, vias 1 -> 0
- net 12V: track 73.2 -> 68.2 mm, vias 1 -> 0
- net Net-(J10-Pin_3): track 63.9 -> 67.9 mm
- net Net-(J10-Pin_1): track 30.9 -> 34.5 mm
- net Net-(D4-A): track 18.0 -> 21.6 mm
- net Net-(D6-K): track 46.5 -> 49.9 mm
- net Net-(J2-Pin_2): track 29.5 -> 32.1 mm, vias 1 -> 0
- net 12VOUT: track 40.3 -> 37.7 mm, vias 1 -> 0
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